Commit message: update
坡脚改前

File: src/simulator/Utils/go2_description/xacro/gazebo.xacro (robot description, xacro)
@@ -15,11 +15,20 @@
     </gazebo>
   </xacro:macro>
-  <xacro:macro name="go2_gazebo">
-    <gazebo>
-      <plugin filename="libgz_ros2_control-system.so"
-              name="gz_ros2_control::GazeboSimROS2ControlPlugin">
-        <parameters>$(find go2_description)/config/ros2_controllers.yaml</parameters>
-      </plugin>
-    </gazebo>
+  <xacro:macro name="go2_gazebo" params="kinematic_mode:=false">
+    <!-- The SCAN demo moves the model through SetEntityPose.  Making it static
+         prevents the physics solver and joint controller from fighting that pose. -->
+    <xacro:if value="${kinematic_mode}">
+      <gazebo>
+        <static>true</static>
+      </gazebo>
+    </xacro:if>
+    <xacro:unless value="${kinematic_mode}">
+      <gazebo>
+        <plugin filename="libgz_ros2_control-system.so"
+                name="gz_ros2_control::GazeboSimROS2ControlPlugin">
+          <parameters>$(find go2_description)/config/ros2_controllers.yaml</parameters>
+        </plugin>
+      </gazebo>
+    </xacro:unless>
     <gazebo reference="imu_link">
       <sensor name="imu_sensor" type="imu">
@@ -30,4 +39,39 @@
       </sensor>
     </gazebo>
+    <gazebo reference="lidar_link">
+      <sensor name="go2_3d_lidar" type="gpu_lidar">
+        <always_on>true</always_on>
+        <visualize>true</visualize>
+        <update_rate>10</update_rate>
+        <topic>/go2/lidar</topic>
+        <gz_frame_id>lidar_link</gz_frame_id>
+        <lidar>
+          <scan>
+            <horizontal>
+              <samples>1024</samples>
+              <resolution>1</resolution>
+              <min_angle>-${pi}</min_angle>
+              <max_angle>${pi}</max_angle>
+            </horizontal>
+            <vertical>
+              <samples>32</samples>
+              <resolution>1</resolution>
+              <min_angle>-${pi / 12.0}</min_angle>
+              <max_angle>${pi / 12.0}</max_angle>
+            </vertical>
+          </scan>
+          <range>
+            <min>0.2</min>
+            <max>30.0</max>
+            <resolution>0.02</resolution>
+          </range>
+          <noise>
+            <type>gaussian</type>
+            <mean>0.0</mean>
+            <stddev>0.01</stddev>
+          </noise>
+        </lidar>
+      </sensor>
+    </gazebo>
     <xacro:go2_foot_contact leg="FL"/>
     <xacro:go2_foot_contact leg="FR"/>

File: src/simulator/Utils/go2_description/xacro/robot.xacro (robot description, xacro)
@@ -3,4 +3,5 @@
     <xacro:arg name="DEBUG" default="false"/>
     <xacro:arg name="use_gazebo" default="true"/>
+    <xacro:arg name="kinematic_mode" default="false"/>
     <xacro:include filename="$(find go2_description)/xacro/const.xacro"/>
     <xacro:include filename="$(find go2_description)/xacro/materials.xacro"/>
@@ -89,4 +90,22 @@
     <link name="front_camera">
     </link>
+    <joint name="lidar_joint" type="fixed">
+        <parent link="trunk"/>
+        <child link="lidar_link"/>
+        <origin rpy="0 0 0" xyz="0 0 0.30"/>
+    </joint>
+    <link name="lidar_link">
+        <visual>
+            <geometry><cylinder radius="0.045" length="0.065"/></geometry>
+            <material name="black"/>
+        </visual>
+        <collision>
+            <geometry><cylinder radius="0.045" length="0.065"/></geometry>
+        </collision>
+        <inertial>
+            <mass value="0.15"/>
+            <inertia ixx="0.0001" ixy="0" ixz="0" iyy="0.0001" iyz="0" izz="0.0001"/>
+        </inertial>
+    </link>
     <!--
     <joint name="load_joint" type="fixed">
@@ -120,6 +139,8 @@
     <xacro:leg name="RL" mirror="1"  mirror_dae="True"   front_hind="-1" front_hind_dae="False" />
     <xacro:if value="$(arg use_gazebo)">
-        <xacro:go2_ros2_control/>
-        <xacro:go2_gazebo/>
+        <xacro:unless value="$(arg kinematic_mode)">
+            <xacro:go2_ros2_control/>
+        </xacro:unless>
+        <xacro:go2_gazebo kinematic_mode="$(arg kinematic_mode)"/>
     </xacro:if>
 </robot>

Commit message: update

File: src/simulator/Utils/go2_description/xacro/gazebo.xacro (robot description, xacro)
@@ -57,5 +57,5 @@
               <samples>32</samples>
               <resolution>1</resolution>
-              <min_angle>-${pi / 12.0}</min_angle>
+              <min_angle>-${pi / 6.0}</min_angle>
               <max_angle>${pi / 12.0}</max_angle>
             </vertical>

File: src/simulator/Utils/go2_description/xacro/robot.xacro (robot description, xacro)
@@ -93,5 +93,6 @@
         <parent link="trunk"/>
         <child link="lidar_link"/>
-        <origin rpy="0 0 0" xyz="0 0 0.30"/>
+        <!-- Keep the sensor just above the trunk to reduce the near-ground blind zone. -->
+        <origin rpy="0 0 0" xyz="0 0 0.12"/>
     </joint>
     <link name="lidar_link">
